Commit message: Modified IMU and encoder msgs to use IMU and Omdometry msgs, added robot description

File: src/robot_description/robot_description.urdf.xacro (robot description, xacro)
@@ -7,5 +7,5 @@
   <xacro:property name="wheel_radius" value="0.03175"/>
   <xacro:property name="wheel_width" value="0.013"/>
-  <xacro:property name="wheel_ygap" value="0.092"/>
+  <xacro:property name="wheel_ygap" value="0.007"/>
   <xacro:property name="wheel_zoff" value="0.0185"/>
   <xacro:property name="wheel_xoff" value="0.088"/>
@@ -42,5 +42,5 @@
       </visual>
     </link>
-    <joint name="${prefix}_joint" type="continuous">
+    <joint name="${prefix}_joint" type="fixed">
       <parent link="base_link"/>
       <child link="${prefix}_link"/>
@@ -67,3 +67,27 @@
     <origin xyz="${caster_xoff} 0.0 ${-(base_height/2)}" rpy="0 0 0"/>
   </joint>
+  <!-- Lidar Link -->
+  <link name="lidar_link">
+  <visual>
+    <geometry>
+    <cylinder radius="0.035" length="0.055" />
+    </geometry>
+    <material name="Gray">
+          <color rgba="0.5 0.5 0.5 1.0"/>
+        </material>
+  </visual>
+  </link>
+  <joint name="lidar_joint" type="fixed">
+    <parent link="base_link"/>
+    <child link="lidar_link"/>
+    <origin xyz="0.05 0 0.055" rpy="0 0 0"/>
+  </joint>
+  <!-- Lidar Link -->
+  <link name="laser">
+  </link>
+  <joint name="laser_joint" type="fixed">
+    <parent link="lidar_link"/>
+    <child link="laser"/>
+    <origin xyz="0 0 0" rpy="0 0 3.14159"/>
+  </joint>
 </robot>

Commit message: Added robot localization package, modified nodes accordingly

File: src/robot_description/robot_description.urdf.xacro (robot description, xacro)
@@ -91,3 +91,10 @@
     <origin xyz="0 0 0" rpy="0 0 3.14159"/>
   </joint>
+  <link name="imu_link">
+  </link>
+  <joint name="imu_joint" type="fixed">
+    <parent link="base_link"/>
+    <child link="imu_link"/>
+    <origin xyz="-0.05 0 0"/>
+  </joint>
 </robot>

Commit message: Updated diff drive, ekf params, launch file with nav

File: src/robot_description/robot_description.urdf.xacro (robot description, xacro)
@@ -5,5 +5,5 @@
   <xacro:property name="base_length" value="0.194"/>
   <xacro:property name="base_height" value="0.067"/>
-  <xacro:property name="wheel_radius" value="0.03175"/>
+  <xacro:property name="wheel_radius" value="0.032499"/>
   <xacro:property name="wheel_width" value="0.013"/>
   <xacro:property name="wheel_ygap" value="0.007"/>
@@ -98,3 +98,22 @@
     <origin xyz="-0.05 0 0"/>
   </joint>
+  <joint name="camera_joint" type="fixed">
+    <parent link="base_link"/>
+    <child link="camera_link"/>
+    <origin xyz="0.1 0 0" rpy="0 0 0"/>
+  </joint>
+  <link name="camera_link">
+    <visual>
+      <geometry>
+        <box size="0.01 0.01 0.01"/>
+      </geometry>
+    </visual>
+  </link>
+  <joint name="camera_optical_joint" type="fixed">
+    <parent link="camera_link"/>
+    <child link="camera_link_optical"/>
+    <origin xyz="0 0 0" rpy="${-pi/2} 0 ${-pi/2}"/>
+  </joint>
+  <link name="camera_link_optical">
+  </link>
 </robot>

Commit message: Update imu driver, motor driver, pid, robot parameters and urdf to new robot chassis

File: src/robot_description/robot_description.urdf.xacro (robot description, xacro)
@@ -2,13 +2,13 @@
 <robot name="pibot" xmlns:xacro="http://ros.org/wiki/xacro">
 <!-- Define robot constants -->
-  <xacro:property name="base_width" value="0.178"/>
-  <xacro:property name="base_length" value="0.194"/>
-  <xacro:property name="base_height" value="0.067"/>
+  <xacro:property name="base_width" value="0.1397"/>
+  <xacro:property name="base_length" value="0.1397"/>
+  <xacro:property name="base_height" value="0.1129"/>
   <xacro:property name="wheel_radius" value="0.032499"/>
-  <xacro:property name="wheel_width" value="0.013"/>
-  <xacro:property name="wheel_ygap" value="0.007"/>
-  <xacro:property name="wheel_zoff" value="0.0185"/>
-  <xacro:property name="wheel_xoff" value="0.088"/>
-  <xacro:property name="caster_xoff" value="0.082"/>
+  <xacro:property name="wheel_width" value="0.025"/>
+  <xacro:property name="wheel_ygap" value="0.015"/>
+  <xacro:property name="wheel_zoff" value="0.07915"/>
+  <xacro:property name="wheel_xoff" value="-0.015"/>
+  <!-- <xacro:property name="caster_xoff" value="-0.085"/> -->
    <!-- Robot Base -->
   <link name="base_link">
@@ -18,14 +18,15 @@
       </geometry>
       <material name="Cyan">
-        <color rgba="0 1.0 1.0 1.0"/>
+        <color rgba="0.0 1.0 1.0 1.0"/>
       </material>
     </visual>
   </link>
   <!-- Robot Footprint -->
+  <!-- z origin ${-(wheel_radius+wheel_zoff+base_height)} -->
   <link name="base_footprint"/>
   <joint name="base_joint" type="fixed">
     <parent link="base_link"/>
     <child link="base_footprint"/>
-    <origin xyz="0.0 0.0 ${-(wheel_radius+wheel_zoff)}" rpy="0 0 0"/>
+    <origin xyz="0.0 0.0 0.0" rpy="0 0 0"/>
   </joint>
     <!-- Wheels -->
@@ -52,8 +53,8 @@
   <xacro:wheel prefix="drivewhl_r" x_reflect="-1" y_reflect="-1" />
     <!-- Caster Wheel -->
-  <link name="front_caster">
+  <!-- <link name="front_caster">
     <visual>
       <geometry>
-        <sphere radius="${(wheel_radius+wheel_zoff-(base_height/2))}"/>
+        <sphere radius="0.020"/>
       </geometry>
       <material name="Cyan">
@@ -66,5 +67,5 @@
     <child link="front_caster"/>
     <origin xyz="${caster_xoff} 0.0 ${-(base_height/2)}" rpy="0 0 0"/>
-  </joint>
+  </joint> -->
   <!-- Lidar Link -->
   <link name="lidar_link">
@@ -81,5 +82,5 @@
     <parent link="base_link"/>
     <child link="lidar_link"/>
-    <origin xyz="0.05 0 0.055" rpy="0 0 0"/>
+    <origin xyz="0.0 0 0.086" rpy="0 0 0"/>
   </joint>
   <!-- Lidar Link -->
