Commit message: Add new launch files for simulation in gazebo, updated urdf files, new rviz config

File: src/robot_description/robot_description.xacro (robot description, xacro)
@@ -4,5 +4,5 @@
   <xacro:property name="base_width" value="0.1397"/>
   <xacro:property name="base_length" value="0.1397"/>
-  <xacro:property name="base_height" value="0.1129"/>
+  <xacro:property name="base_height" value="0.1194"/>
   <xacro:property name="wheel_radius" value="0.032499"/>
   <xacro:property name="wheel_width" value="0.025"/>
@@ -10,5 +10,5 @@
   <xacro:property name="wheel_zoff" value="0.07915"/>
   <xacro:property name="wheel_xoff" value="-0.015"/>
-  <!-- <xacro:property name="caster_xoff" value="-0.085"/> -->
+  <xacro:property name="caster_xoff" value="-0.085"/>
    <!-- Robot Base -->
   <link name="base_link">
@@ -24,9 +24,31 @@
   <!-- Robot Footprint -->
   <!-- z origin ${-(wheel_radius+wheel_zoff+base_height)} -->
-  <link name="base_footprint"/>
+  <link name="base_footprint">
+  </link>
   <joint name="base_joint" type="fixed">
     <parent link="base_link"/>
     <child link="base_footprint"/>
-    <origin xyz="0.0 0.0 0.0" rpy="0 0 0"/>
+    <origin xyz="0.0 0.0 -${(base_height/2-wheel_radius+wheel_zoff)}" rpy="0 0 0"/>
+  </joint>
+  <xacro:macro name="box_inertia" params="m w h d">
+    <inertial>
+      <origin xyz="0 0 ${-(base_height/2)}" rpy="0 0 0"/>
+      <mass value="${m}"/>
+      <inertia ixx="${(m/12) * (h*h + d*d)}" ixy="0.0" ixz="0.0" iyy="${(m/12) * (w*w + d*d)}" iyz="0.0" izz="${(m/12) * (w*w + h*h)}"/>
+    </inertial>
+  </xacro:macro>
+  <link name="chassis">
+  <collision>
+      <origin xyz="0 0 0" rpy="0 0 0"/>
+      <geometry>
+        <box size="${base_length} ${base_width} ${base_height}"/>
+      </geometry>
+    </collision>
+    <xacro:box_inertia m="6" w="${base_width}" d="${base_length}" h="${base_height}"/>
+  </link>
+  <joint name="chassis_joint" type="fixed">
+    <parent link="base_link"/>
+    <child link="chassis"/>
+    <origin xyz="0 0 0" rpy="0 0 0"/>
   </joint>
     <!-- Wheels -->
@@ -42,6 +64,21 @@
         </material>
       </visual>
+      <collision>
+        <origin xyz="0 0 0" rpy="${pi/2} 0 0"/>
+        <geometry>
+            <cylinder radius="${wheel_radius}" length="${wheel_width}"/>
+        </geometry>
+      </collision>
+      <inertial>
+      <mass value="0.5"/>
+      <inertia ixx="${(1/12) * 0.1 * (3 * wheel_radius + wheel_width*wheel_width)}"
+               ixy="0.0"
+               ixz="0.0"
+               iyy="${(1/12) * 0.1 * (3 * wheel_radius + wheel_width*wheel_width)}"
+               iyz="0.0"
+               izz="${(1/12) * 0.1 * (3 * wheel_radius + wheel_width*wheel_width)}"/>
+      </inertial>
     </link>
-    <joint name="${prefix}_joint" type="fixed">
+    <joint name="${prefix}_joint" type="continuous">
       <parent link="base_link"/>
       <child link="${prefix}_link"/>
@@ -53,19 +90,36 @@
   <xacro:wheel prefix="drivewhl_r" x_reflect="-1" y_reflect="-1" />
     <!-- Caster Wheel -->
-  <!-- <link name="front_caster">
+  <link name="rear_caster">
     <visual>
       <geometry>
         <sphere radius="0.020"/>
       </geometry>
-      <material name="Cyan">
-        <color rgba="0 1.0 1.0 1.0"/>
+      <material name="White">
+        <color rgba="1.0 1.0 1.0 1.0"/>
       </material>
     </visual>
+    <collision>
+      <origin xyz="0 0 0" rpy="0 0 0"/>
+      <geometry>
+        <sphere radius="0.020"/>
+      </geometry>
+    </collision>
+    <inertial>
+      <mass value="1.0"/>
+      <inertia
+        ixx="${(2/5 * 0.01 * (0.02 * 0.02))}"
+        ixy="0.0"
+        ixz="0.0"
+        iyy="${(2/5 * 0.01 * (0.02 * 0.02))}"
+        iyz="0.0"
+        izz="${(2/5 * 0.01 * (0.02 * 0.02))}"
+      />
+    </inertial>
   </link>
   <joint name="caster_joint" type="fixed">
     <parent link="base_link"/>
-    <child link="front_caster"/>
-    <origin xyz="${caster_xoff} 0.0 ${-(base_height/2)}" rpy="0 0 0"/>
-  </joint> -->
+    <child link="rear_caster"/>
+    <origin xyz="${caster_xoff} 0.0 ${-(base_height/2 + wheel_radius)}" rpy="0 0 0"/>
+  </joint>
   <!-- Lidar Link -->
   <link name="lidar_link">

Commit message: update parameters for new chassis and video stream

File: src/robot_description/robot_description.xacro (robot description, xacro)
@@ -2,13 +2,13 @@
 <robot name="pibot" xmlns:xacro="http://ros.org/wiki/xacro">
 <!-- Define robot constants -->
-  <xacro:property name="base_width" value="0.1397"/>
-  <xacro:property name="base_length" value="0.1397"/>
-  <xacro:property name="base_height" value="0.1194"/>
-  <xacro:property name="wheel_radius" value="0.032499"/>
-  <xacro:property name="wheel_width" value="0.025"/>
-  <xacro:property name="wheel_ygap" value="0.015"/>
+  <xacro:property name="base_width" value="0.2794"/>
+  <xacro:property name="base_length" value="0.4318"/>
+  <xacro:property name="base_height" value="0.17145"/>
+  <xacro:property name="wheel_radius" value="0.06604"/>
+  <xacro:property name="wheel_width" value="0.066675"/>
+  <xacro:property name="wheel_ygap" value="0.03"/>
   <xacro:property name="wheel_zoff" value="0.07915"/>
-  <xacro:property name="wheel_xoff" value="-0.015"/>
-  <xacro:property name="caster_xoff" value="-0.085"/>
+  <xacro:property name="wheel_xoff" value="-0.08255"/>
+  <xacro:property name="caster_xoff" value="-0.1555"/>
    <!-- Robot Base -->
   <link name="base_link">
@@ -80,5 +80,6 @@
       </inertial>
     </link>
-    <joint name="${prefix}_joint" type="continuous">
+<!-- change type to fixed for rviz -->
+    <joint name="${prefix}_joint" type="fixed">
       <parent link="base_link"/>
       <child link="${prefix}_link"/>
@@ -93,5 +94,5 @@
     <visual>
       <geometry>
-        <sphere radius="0.020"/>
+        <sphere radius="0.0254"/>
       </geometry>
       <material name="White">
@@ -120,5 +121,5 @@
     <parent link="base_link"/>
     <child link="rear_caster"/>
-    <origin xyz="${caster_xoff} 0.0 ${-(base_height/2 + wheel_radius)}" rpy="0 0 0"/>
+    <origin xyz="${caster_xoff} 0.0 ${-(base_height/2 + 0.025)}" rpy="0 0 0"/>
   </joint>
   <!-- Lidar Link -->
@@ -136,5 +137,5 @@
     <parent link="base_link"/>
     <child link="lidar_link"/>
-    <origin xyz="0.0 0 0.086" rpy="0 0 0"/>
+    <origin xyz="0.1365 0 0.11" rpy="0 0 0"/>
   </joint>
   <!-- Lidar Link -->
